Commit message: Update pyramid.urdf.xacro

File: q2/pyramid.urdf.xacro (robot description, xacro)
@@ -19,5 +19,5 @@
       <geometry>
         <!-- <box size="0.1 0.1 0.1"/> -->
-        <mesh filename="package://pcl_task/meshes/illuminati_pyramid.dae/>
+        <mesh filename="package://pcl_task/meshes/illuminati_pyramid.dae"/>
       </geometry>
     </visual>
